File: Constant Current Load/load.brd (EAGLE design)
At the start: 46 parts, among them IC1 LM324P, J1 6_PIN_SERIAL_CABLEPTH

Commit message: Starting work on double sided board
Parts:
- removed VREGOUT2: 10uf, resistor:E2,5-6
- R12: value 22k -> 15k
Connections:
- net +12V: no longer VREGOUT2.+
- net GND: no longer VREGOUT2.-
Routing:
- net +12V: track 115.2 -> 112.9 mm
Changed lines of the file:
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@@
 <?xml version="1.0" encoding="utf-8"?>
 <!DOCTYPE eagle SYSTEM "eagle.dtd">
-<eagle version="8.1.1">
+<eagle version="8.2.2">
 <drawing>
 <settings>
@@
 <element name="C2" library="rcl" package="E2,5-6E" value="10u" x="-119.38" y="-113.792" rot="R90"/>
 <element name="R11" library="rcl" package="RTRIM64W" value="100k" x="-74.422" y="-121.92" rot="R270"/>
-<element name="R12" library="resistor" package="0207/7" value="22k" x="-35.56" y="-92.964" rot="R180"/>
+<element name="R12" library="resistor" package="0207/7" value="15k" x="-35.56" y="-92.964" rot="R180"/>
 <element name="AREF_SET" library="rcl" package="RTRIM64W" value="100k" x="-91.694" y="-117.856" rot="R90"/>
 <element name="5VREG" library="SparkFun-IC-Power" package="TO-252" value="7805" x="-39.37" y="-81.28" rot="MR270">
@@
 <attribute name="PROD_ID" value="VREG-12370" x="-99.314" y="-81.026" size="1.778" layer="28" rot="MR270" display="off"/>
 </element>
-<element name="VREGOUT2" library="resistor" package="E2,5-6" value="10uf" x="-52.324" y="-79.502"/>
 </elements>
 <signals>
@@
 <contactref element="5VREG" pad="3"/>
 <contactref element="7812" pad="3"/>
-<contactref element="VREGOUT2" pad="-"/>
+<wire x1="-112.014" y1="-133.858" x2="-115.824" y2="-133.858" width="0" layer="19" extent="1-1"/>
+<wire x1="-108.204" y1="-133.858" x2="-112.014" y2="-133.858" width="0" layer="19" extent="1-1"/>
+<wire x1="-104.394" y1="-133.858" x2="-108.204" y2="-133.858" width="0" layer="19" extent="1-1"/>
+<wire x1="-100.584" y1="-133.858" x2="-104.394" y2="-133.858" width="0" layer="19" extent="1-1"/>
+<wire x1="-96.774" y1="-133.858" x2="-100.584" y2="-133.858" width="0" layer="19" extent="1-1"/>
+<wire x1="-92.964" y1="-133.858" x2="-96.774" y2="-133.858" width="0" layer="19" extent="1-1"/>
+<wire x1="-89.154" y1="-133.858" x2="-92.964" y2="-133.858" width="0" layer="19" extent="1-1"/>
+<wire x1="-85.344" y1="-133.858" x2="-89.154" y2="-133.858" width="0" layer="19" extent="1-1"/>
+<wire x1="-81.534" y1="-133.858" x2="-85.344" y2="-133.858" width="0" layer="19" extent="1-1"/>
+<wire x1="-74.168" y1="-134.874" x2="-81.534" y2="-133.858" width="0" layer="19" extent="1-1"/>
+<wire x1="-70.866" y1="-126.492" x2="-74.168" y2="-127.254" width="0" layer="19" extent="1-1"/>
+<wire x1="-71.882" y1="-123.19" x2="-70.866" y2="-126.492" width="0" layer="19" extent="1-1"/>
+<wire x1="-74.168" y1="-117.348" x2="-71.882" y2="-123.19" width="0" layer="19" extent="1-1"/>
+<wire x1="-124.46" y1="-127" x2="-115.824" y2="-133.858" width="0" layer="19" extent="1-1"/>
+<wire x1="-119.38" y1="-112.522" x2="-124.46" y2="-120.904" width="0" layer="19" extent="1-1"/>
+<wire x1="-122.682" y1="-105.41" x2="-119.38" y2="-112.522" width="0" layer="19" extent="1-1"/>
+<wire x1="-123.19" y1="-102.87" x2="-122.682" y2="-105.41" width="0" layer="19" extent="1-1"/>
+<wire x1="-125.984" y1="-95.504" x2="-123.19" y2="-93.98" width="0" layer="19" extent="1-1"/>
+<wire x1="-102.616" y1="-103.378" x2="-109.982" y2="-105.41" width="0" layer="19" extent="1-1"/>
+<wire x1="-87.884" y1="-103.378" x2="-91.694" y2="-106.172" width="0" layer="19" extent="1-1"/>
+<wire x1="-104.39" y1="-97.53" x2="-102.616" y2="-103.378" width="0" layer="19" extent="1-1"/>
+<wire x1="-89.154" y1="-113.792" x2="-91.694" y2="-107.95" width="0" layer="19" extent="16-16"/>
+<wire x1="-89.154" y1="-116.586" x2="-89.154" y2="-113.792" width="0" layer="19" extent="1-1"/>
+<wire x1="-104.14" y1="-90.17" x2="-104.39" y2="-97.53" width="0" layer="19" extent="1-1"/>
+<wire x1="-126.874" y1="-86.9" x2="-123.19" y2="-93.98" width="0" layer="19" extent="1-1"/>
+<wire x1="-122.174" y1="-83.9" x2="-126.874" y2="-86.9" width="0" layer="19" extent="1-1"/>
+<wire x1="-114.55" y1="-97.53" x2="-109.982" y2="-105.41" width="0" layer="19" extent="1-1"/>
+<wire x1="-101.814" y1="-81.026" x2="-104.14" y2="-90.17" width="0" layer="19" extent="16-16"/>
+<wire x1="-108.2294" y1="-80.518" x2="-101.814" y2="-81.026" width="0" layer="19" extent="16-16"/>
+<wire x1="-91.44" y1="-80.772" x2="-101.814" y2="-81.026" width="0" layer="19" extent="16-16"/>
+<wire x1="-87.376" y1="-78.994" x2="-91.44" y2="-80.772" width="0" layer="19" extent="1-1"/>
+<wire x1="-76.962" y1="-84.034" x2="-87.376" y2="-78.994" width="0" layer="19" extent="1-1"/>
+<wire x1="-71.374" y1="-88.646" x2="-76.962" y2="-84.034" width="0" layer="19" extent="1-1"/>
+<wire x1="-68.2" y1="-86.9" x2="-71.374" y2="-88.646" width="0" layer="19" extent="1-1"/>
+<wire x1="-63.5" y1="-83.9" x2="-68.2" y2="-86.9" width="0" layer="19" extent="1-1"/>
+<wire x1="-55.8292" y1="-84.0994" x2="-63.5" y2="-83.9" width="0" layer="19" extent="1-1"/>
+<wire x1="-49.3268" y1="-84.0994" x2="-55.8292" y2="-84.0994" width="0" layer="19" extent="1-1"/>
+<wire x1="-41.87" y1="-81.28" x2="-49.3268" y2="-84.0994" width="0" layer="19" extent="16-16"/>
+<wire x1="-37.592" y1="-89.916" x2="-41.87" y2="-81.28" width="0" layer="19" extent="16-16"/>
+<wire x1="-39.116" y1="-97.536" x2="-37.592" y2="-89.916" width="0" layer="19" extent="1-1"/>
+<wire x1="-70.358" y1="-100.076" x2="-71.374" y2="-88.646" width="0" layer="19" extent="1-1"/>
+<wire x1="-73.406" y1="-100.076" x2="-70.358" y2="-100.076" width="0" layer="19" extent="1-1"/>
+<wire x1="-34.29" y1="-110.49" x2="-39.116" y2="-97.536" width="0" layer="19" extent="1-1"/>
+<wire x1="-54.864" y1="-114.554" x2="-71.882" y2="-123.19" width="0" layer="19" extent="1-1"/>
+<wire x1="-52.324" y1="-119.888" x2="-54.864" y2="-114.554" width="0" layer="19" extent="1-1"/>
 </signal>
 <signal name="V_ACC_RESISTOR">
@@
 <wire x1="-36.354" y1="-77.216" x2="-34.57" y2="-79" width="0.4064" layer="16"/>
 <wire x1="-72.644" y1="-82.296" x2="-67.564" y2="-77.216" width="0.4064" layer="16"/>
-<contactref element="VREGOUT2" pad="+"/>
-<wire x1="-53.594" y1="-79.502" x2="-53.594" y2="-77.216" width="0.4064" layer="16"/>
 </signal>
 <signal name="V+">

Commit message: Replaced through hole with smd
Parts:
- C1POWER, VREGIN1: value .1uf -> .1uF; device rcl:C025-025X050 -> rcl:C0805K
- C3, C4: value 22pf -> 22pF; device rcl:C025-025X050 -> rcl:C0805K
- LCD_BAK_RES, LCD_POW_RES, RESETPULLUP: device rcl:0204/7 -> resistor:M0805
- PULLDOWN0: value 30k -> 30K; device rcl:0204/7 -> resistor:M0805
- PULLDOWN1: value 20k -> 20K; device rcl:0204/7 -> resistor:M0805
- R12: value 15k -> 15K; device resistor:0207/7 -> resistor:M0805
- RESETCAP: value .1uf -> 0.33µF; device rcl:C025-025X050 -> rcl:C0805K
- VREGIN2: device rcl:C025-025X050 -> rcl:C0805K
- moved LCD_POW_RES 448.4 mm to (320.0, 19.1), turned to 90 degrees
- moved C4 430.8 mm to (310.4, 20.6)
- moved C1POWER 300.4 mm to (201.2, 5.60), turned to 90 degrees
- moved RESETCAP 295.1 mm to (216.4, 21.1), turned to 90 degrees
- moved VREGIN1 282.7 mm to (178.3, 21.1), turned to 90 degrees
- moved LCD_BAK_RES 266.3 mm to (165.6, 21.1)
- moved VREGIN2 257.8 mm to (191.0, 21.1), turned to 90 degrees
- moved C3 220.3 mm to (105.7, 3.06)
- moved PULLDOWN0 206.5 mm to (109.2, 10.5), turned to 90 degrees
- moved RESETPULLUP 185.4 mm to (97.3, 23.2), turned to 90 degrees
- moved PULLDOWN1 177.8 mm to (78.0, 1.84)
- moved R12 115.1 mm to (4.83, 14.8), turned to 90 degrees
Routing:
- net 12V_I/P_TEST: track 103.3 -> 0.00 mm
- net +12V: track 112.9 -> 27.6 mm
- net GND: track 69.8 -> 15.2 mm, vias 12 -> 0
- net V+: track 105.3 -> 52.5 mm
- net DTR: track 39.2 -> 0.00 mm
- net +5V: track 201.9 -> 184.7 mm
- net N$9: track 13.5 -> 0.00 mm
- net 12V_JACK_INPUT: track 51.9 -> 38.8 mm
- net CRYSTAL2: track 9.91 -> 4.43 mm
- net RESET: track 46.3 -> 41.3 mm
- net CRYSTAL1: track 10.1 -> 6.82 mm
- net N$7: track 7.39 -> 4.60 mm
- net N$14: track 6.33 -> 4.30 mm

Commit message: Routed the pcb v1
Parts:
- moved LCD_POW_RES 289.4 mm to (31.8, 45.5), turned to 0 degrees
- moved C4 269.4 mm to (42.2, 46.2), turned to 270 degrees
- moved 7812 212.9 mm to (54.9, 65.8), flipped to the top, turned to 0 degrees
- moved VREGOUT1 211.3 mm to (63.0, 62.2)
- moved AREF_SET 206.6 mm to (53.1, 29.5)
- moved C2 206.6 mm to (25.4, 33.5)
- moved CRYSTAL 206.6 mm to (49.5, 45.2)
- moved CURRENT_SET_RES 206.6 mm to (109.2, 39.4)
- moved IC1 206.6 mm to (89.9, 36.6)
- moved J1 206.6 mm to (86.6, 20.8)
- moved JP1 206.6 mm to (48.3, 57.9)
- moved LCD1 206.6 mm to (62.2, 34.3)
- moved LCD_CONTRAST 206.6 mm to (38.1, 55.9)
- moved LOAD_JACK 206.6 mm to (22.6, 71.1)
- moved MOSFET 206.6 mm to (16.8, 37.8)
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Routing:
- net GATE_V: track 207.0 -> 144.5 mm, vias 0 -> 2
- net 12V_I/P_TEST: track 0.00 -> 45.6 mm, vias 0 -> 3
- net +12V: track 27.6 -> 63.9 mm, vias 0 -> 2
- net V+: track 52.5 -> 80.7 mm
- net +5V: track 184.7 -> 165.1 mm, vias 0 -> 2
- net RESET: track 41.3 -> 59.6 mm
- net 12V_JACK_INPUT: track 38.8 -> 25.9 mm
- net N$9: track 0.00 -> 12.9 mm
- net RX: track 39.3 -> 27.4 mm, vias 0 -> 2
- net LCD_D4: track 24.8 -> 16.6 mm
- net DTR: track 0.00 -> 5.62 mm
- net CRYSTAL2: track 4.43 -> 9.39 mm
- net LCD_E: track 12.7 -> 8.64 mm, vias 0 -> 1
- net CRYSTAL1: track 6.82 -> 9.60 mm
- net V+_DIVIDED: track 62.4 -> 60.0 mm
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- added copper zone on layer 1, net GND

Commit message: Still working
Parts:
- added J2: AVR_SPI_PROG_5X2PTH2, SparkFun-Connectors:2X5-SHROUDED
- added VREGOUT2: 10uf, resistor:E2,5-6
- BACKLIGHT_E: value bklight enable -> (none)
- moved MOSFET 8.89 mm to (7.87, 37.8)
- renumbered JP1 to BACKLIGHT_E, R11 to GATE_V
Connections:
- removed net 12V_I/P_TEST: PULLDOWN0.1, PULLDOWN1.2, UC.19
- removed net D11: UC.17
- removed net D12: UC.18
- new net MISO: J2.9, UC.18
- new net MOSI: J2.1, UC.17
- new net PB5/SCK: J2.7, PULLDOWN0.1, PULLDOWN1.2, UC.19
- new net VCC: J2.2
- net 12V_JACK_INPUT: now also VREGOUT2.+
- net GND: now also J2.10, J2.4, J2.6, J2.8, VREGOUT2.-
- net RESET: now also J2.5
Routing:
- net RESET: track 59.6 -> 175.2 mm, vias 0 -> 3
- net PB5/SCK: track 0.00 -> 97.0 mm, vias 0 -> 3
- net MISO: track 0.00 -> 46.4 mm
- net 12V_I/P_TEST: track 45.6 -> 0.00 mm, vias 3 -> 0
- net MOSI: track 0.00 -> 32.4 mm
- net N$8: track 366.3 -> 391.7 mm
- net V+: track 80.7 -> 96.2 mm
- net V_ACC_RESISTOR: track 144.8 -> 158.0 mm
- net 12V_JACK_INPUT: track 25.9 -> 29.0 mm
- net GATE_V: track 144.5 -> 147.4 mm
- net LCD_E: vias 1 -> 0
- net LCD_RS: vias 1 -> 0
