File: Constant Current Load/load.brd (EAGLE design)
At the start: 47 parts, among them IC1 LM324P, J1 6_PIN_SERIAL_CABLEPTH, J2 AVR_SPI_PROG_5X2PTH2

Commit message: Still working
Parts:
- removed POW_SLECTION_JUMPER: (no value), pinhead:1X03
- added JP1, POW_SELECT: (no value), pinhead:1X03
- AREF_SET, CURRENT_SET_RES, GATE_V, LCD_CONTRAST, V+_DIVIDER: device rcl:RTRIM64W -> pot:S64W
- moved GATE_V 55.7 mm to (16.0, 37.3), turned to 0 degrees
- moved AREF_SET 39.7 mm to (16.0, 43.7), turned to 0 degrees
- moved R12 9.33 mm to (95.8, 46.3)
- moved C2 6.14 mm to (27.9, 39.1)
- moved VREGOUT2 4.83 mm to (69.8, 57.4)
- moved VREGOUT1 4.83 mm to (63.0, 57.4)
- moved R1 3.59 mm to (54.4, 22.4)
- moved R10 3.59 mm to (35.3, 22.4)
- moved R2 3.59 mm to (50.5, 22.4)
- moved R3 3.59 mm to (58.2, 22.4)
- moved R4 3.59 mm to (46.7, 22.4)
- moved R5 3.59 mm to (31.5, 22.4)
- moved R6 3.59 mm to (42.9, 22.4)
- moved R7 3.59 mm to (65.8, 22.4)
- moved R8 3.59 mm to (39.1, 22.4)
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- renumbered SUPPLY_JACK to 12V
Connections:
- removed net VCC: J2.2
- new net N$2: 7812.1, JP1.1, VREGIN1.1
- net +12V: now also POW_SELECT.2; no longer POW_SLECTION_JUMPER.2
- net +5V: now also AREF_SET.A, J2.2, LCD_CONTRAST.E; no longer AREF_SET.3, LCD_CONTRAST.3
- net 12V_JACK_INPUT: now also POW_SELECT.1; no longer POW_SLECTION_JUMPER.1
- net 12V_REG_O/P: now also POW_SELECT.3; no longer POW_SLECTION_JUMPER.3
- net A2: now also GATE_V.S; no longer GATE_V.2
- net AREF: now also AREF_SET.S; no longer AREF_SET.2
- net GATE_V: now also GATE_V.A; no longer GATE_V.1
- net GND: now also AREF_SET.E, CURRENT_SET_RES.A, GATE_V.E, LCD_CONTRAST.A, V+_DIVIDER.E; no longer AREF_SET.1, CURRENT_SET_RES.1, GATE_V.3, LCD_CONTRAST.1, V+_DIVIDER.3
- net N$1: now also CURRENT_SET_RES.S; no longer CURRENT_SET_RES.2
- net N$6: now also LCD_CONTRAST.S; no longer LCD_CONTRAST.2
- net N$9: now also CURRENT_SET_RES.E; no longer CURRENT_SET_RES.3
- net V+: now also JP1.2, V+_DIVIDER.A; no longer 7812.1, V+_DIVIDER.1, VREGIN1.1
- net V+_DIVIDED: now also V+_DIVIDER.S; no longer V+_DIVIDER.2
Routing:
- net +5V: track 165.1 -> 244.9 mm, vias 2 -> 3
- net AREF: track 2.79 -> 44.2 mm, vias 0 -> 1
- net A2: track 12.3 -> 51.1 mm, vias 0 -> 1
- net N$2: track 0.00 -> 23.4 mm, vias 0 -> 1
- net 12V_REG_O/P: track 10.2 -> 27.6 mm
- net V_ACC_RESISTOR: track 158.0 -> 141.8 mm, vias 2 -> 1
- net GND: track 15.2 -> 0.00 mm
- net RX: track 27.4 -> 35.9 mm, vias 2 -> 3
- net RESET: track 175.2 -> 168.1 mm, vias 3 -> 1
- net 12V_JACK_INPUT: track 29.0 -> 33.6 mm
- net PB5/SCK: track 97.0 -> 101.5 mm, vias 3 -> 6
- net TX: track 33.4 -> 37.4 mm, vias 0 -> 1
- net DTR: track 5.62 -> 9.05 mm
- net +12V: track 63.9 -> 66.7 mm
- net N$9: track 12.9 -> 15.4 mm
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
Commit message: Still working
Parts:
- removed LCD_BAK_RES: 220, resistor:M0805
- added BACK_RES: 220, resistor:M0805
- added C1POWER1, C1POWER2: .1uF, rcl:C0805K
- added U$1: (no value), heatsink:SK129-HOLE
- moved CURRENT_SET_RES 12.1 mm to (106.7, 51.3), turned to 0 degrees
- moved MOSFET 6.35 mm to (1.52, 37.8)
- moved C1POWER 4.57 mm to (35.3, 46.4)
- renumbered BACKLIGHT_E to BACKLIGHT, LCD_CONTRAST to CONTRAST
Connections:
- net +5V: now also C1POWER1.1
- net AREF: now also C1POWER2.1
- net GND: now also BACK_RES.1, C1POWER1.2, C1POWER2.2; no longer LCD_BAK_RES.1
- net N$14: now also BACK_RES.2; no longer LCD_BAK_RES.2
Routing:
- net N$8: track 391.7 -> 0.00 mm
- net +5V: track 244.9 -> 260.7 mm
- net V+: track 97.7 -> 111.8 mm
- net GATE_V: track 145.8 -> 152.2 mm
- net V_ACC_RESISTOR: track 141.8 -> 148.1 mm
- net N$1: track 22.5 -> 25.1 mm
- net AREF: track 44.2 -> 46.0 mm
- net V+_DIVIDED: track 58.5 -> 59.7 mm
- net PB5/SCK: track 101.5 -> 100.9 mm
Other:
- board outline added: 145 x 63.5 mm

Commit message: Complete I guess
Parts:
- removed CURRENT_SET_RES: 10k, pot:S64W
- added CURRENT_SET: 10k, pot:S64W
- 7805: value 7805 -> 5V
- renumbered 5VREG to 7805, AREF_SET to AREF, BACK_RES to R15, C1POWER to C9, C1POWER1 to C8, C1POWER2 to C11, CONTRAST to CONT, IC1 to OPAMP, J1 to FTDI, J2 to ASP, JP1 to V+TO12, LCD1 to LCD, LCD_POW_RES to R16, PULLDOWN0 to R14, PULLDOWN1 to R13, RESETCAP to C10, RESETPULLUP to R17, U$1 to HEATSINK, UC to ATMEGA328P, V+_DIVIDER to V+, VREGIN1 to C6, VREGIN2 to C13, VREGOUT to C12, VREGOUT1 to C5, VREGOUT2 to C7, X1 to LOAD
Connections:
- net GND: now also CURRENT_SET.A; no longer CURRENT_SET_RES.A
- net N$1: now also CURRENT_SET.S; no longer CURRENT_SET_RES.S
- net N$9: now also CURRENT_SET.E; no longer CURRENT_SET_RES.E
Routing:
- net N$1: track 25.1 -> 17.8 mm
- net N$9: track 15.1 -> 12.6 mm
Other:
- board text added: "DTR"
- board text added: "GND"

Commit message: Before moving HS and Pot
Other:
- board text added: "+"
- board text added: "-"
Changed lines of the file:
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@@
 <text x="73.66" y="14.732" size="1.016" layer="25">GND</text>
 <text x="86.614" y="14.732" size="1.016" layer="25">DTR</text>
+<text x="29.464" y="70.104" size="1.778" layer="25">+</text>
+<text x="36.83" y="70.104" size="1.778" layer="25">-</text>
 </plain>
 <attributes>
@@
 <attribute name="MF" value="" x="34.036" y="66.802" size="1.778" layer="27" display="off"/>
 <attribute name="MPN" value="" x="34.036" y="66.802" size="1.778" layer="27" display="off"/>
-<attribute name="NAME" x="28.956" y="70.358" size="1.27" layer="25" ratio="10"/>
+<attribute name="NAME" x="31.496" y="70.104" size="1.27" layer="25" ratio="10"/>
 <attribute name="OC_FARNELL" value="unknown" x="34.036" y="66.802" size="1.778" layer="27" display="off"/>
 <attribute name="OC_NEWARK" value="unknown" x="34.036" y="66.802" size="1.778" layer="27" display="off"/>
@@
 <signal name="N$5">
 </signal>
-<signal name="N$3">
-</signal>
 <signal name="N$4">

Commit message: Final
Parts:
- moved CURRENT_SET 58.2 mm to (64.5, 4.83), turned to 0 degrees
- moved HEATSINK 53.1 mm to (33.8, -1.52), turned to 0 degrees
- moved MOSFET 48.4 mm to (33.8, 1.78), turned to 180 degrees
- moved R5 34.3 mm to (65.8, 22.1), turned to 270 degrees
- moved R7 34.3 mm to (31.5, 22.1), turned to 270 degrees
- moved R10 26.7 mm to (62.0, 22.1), turned to 270 degrees
- moved R9 26.7 mm to (35.3, 22.1), turned to 270 degrees
- moved R3 19.1 mm to (39.1, 22.1), turned to 270 degrees
- moved R8 19.1 mm to (58.2, 22.1), turned to 270 degrees
- moved C2 14.2 mm to (25.7, 25.1)
- moved R1 11.4 mm to (42.9, 22.1), turned to 270 degrees
- moved R6 11.4 mm to (54.4, 22.1), turned to 270 degrees
- moved 7805 11.4 mm to (90.2, 65.8)
- moved RESET 7.94 mm to (98.3, 66.0), turned to 270 degrees
- moved LOAD_JACK 6.35 mm to (16.3, 71.1)
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Routing:
- net N$9: track 12.6 -> 90.7 mm
- net N$1: track 17.8 -> 87.9 mm
- net V+: track 111.8 -> 169.9 mm
- net +5V: track 260.7 -> 230.9 mm
- net GATE_V: track 152.2 -> 176.5 mm, vias 1 -> 3
- net RESET: track 168.1 -> 181.0 mm, vias 1 -> 3
- net V_ACC_RESISTOR: track 148.1 -> 139.9 mm
- net +12V: track 66.6 -> 63.5 mm
Other:
- board size 145 x 63.5 mm -> 98.3 x 89.2 mm
- board text added: "12/Sep/17"
- board text added: "Chirag Shah"
- board text added: "Constant Current Load"
