File: Constant Current Load/load.sch (EAGLE design)
At the start: 46 parts, among them IC1 LM324P, J1 6_PIN_SERIAL_CABLEPTH

Commit message: Starting work on double sided board
Parts:
- removed VREGOUT2: 10uf, resistor:CPOL-EUE2.5-6
- R12: value 22k -> 15k
Connections:
- net +12V: no longer VREGOUT2.+
- net GND: no longer VREGOUT2.-
Other:
- moved on the sheet: MOSFET
Changed lines of the file:
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@@
 <?xml version="1.0" encoding="utf-8"?>
 <!DOCTYPE eagle SYSTEM "eagle.dtd">
-<eagle version="8.1.1">
+<eagle version="8.2.2">
 <drawing>
 <settings>
@@
 <part name="R11" library="rcl" deviceset="R-TRIMM" device="64W" value="100k"/>
 <part name="GND9" library="supply1" deviceset="GND" device=""/>
-<part name="R12" library="resistor" deviceset="R-EU_" device="0207/7" value="22k"/>
+<part name="R12" library="resistor" deviceset="R-EU_" device="0207/7" value="15k"/>
 <part name="AREF_SET" library="rcl" deviceset="R-TRIMM" device="64W" value="100k"/>
 <part name="GND23" library="supply1" deviceset="GND" device=""/>
 <part name="5VREG" library="SparkFun-IC-Power" deviceset="V_REG_78XX" device="7812" value="7805"/>
 <part name="7812" library="SparkFun-IC-Power" deviceset="V_REG_78XX" device="7812" value="+12v"/>
-<part name="VREGOUT2" library="resistor" deviceset="CPOL-EU" device="E2.5-6" value="10uf"/>
 </parts>
 <sheets>
@@
 <instance part="R9" gate="G$1" x="96.52" y="45.72" rot="R90"/>
 <instance part="R10" gate="G$1" x="99.06" y="45.72" rot="R90"/>
-<instance part="MOSFET" gate="NMOS" x="83.82" y="71.12"/>
+<instance part="MOSFET" gate="NMOS" x="86.36" y="71.12"/>
 <instance part="IC1" gate="A" x="40.64" y="68.58"/>
 <instance part="GND1" gate="1" x="38.1" y="55.88"/>
@@
 <pinref part="IC1" gate="A" pin="OUT"/>
 <pinref part="MOSFET" gate="NMOS" pin="G"/>
-<wire x1="48.26" y1="68.58" x2="78.74" y2="68.58" width="0.1524" layer="91"/>
+<wire x1="48.26" y1="68.58" x2="81.28" y2="68.58" width="0.1524" layer="91"/>
 <label x="55.88" y="71.12" size="1.778" layer="95"/>
 </segment>
@@
 <junction x="99.06" y="50.8"/>
 <pinref part="MOSFET" gate="NMOS" pin="S"/>
-<wire x1="86.36" y1="66.04" x2="88.9" y2="55.88" width="0.1524" layer="91"/>
+<wire x1="88.9" y1="66.04" x2="88.9" y2="55.88" width="0.1524" layer="91"/>
 <wire x1="88.9" y1="55.88" x2="88.9" y2="50.8" width="0.1524" layer="91"/>
 <wire x1="63.5" y1="55.88" x2="88.9" y2="55.88" width="0.1524" layer="91"/>
@@
 <segment>
 <pinref part="MOSFET" gate="NMOS" pin="D"/>
-<wire x1="86.36" y1="76.2" x2="88.9" y2="86.36" width="0.1524" layer="91"/>
+<wire x1="88.9" y1="76.2" x2="88.9" y2="86.36" width="0.1524" layer="91"/>
 <pinref part="P+3" gate="1" pin="V+"/>
 <wire x1="88.9" y1="86.36" x2="88.9" y2="88.9" width="0.1524" layer="91"/>
@@
 <attribute name="VALUE" x="71.12" y="146.05" size="1.778" layer="96"/>
 </instance>
-<instance part="VREGOUT2" gate="G$1" x="45.72" y="139.7" smashed="yes">
-<attribute name="NAME" x="50.3174" y="135.763" size="1.778" layer="95" rot="R90"/>
-<attribute name="VALUE" x="52.8574" y="135.763" size="1.778" layer="96" rot="R90"/>
-</instance>
 </instances>
 <busses>
@@
 <wire x1="71.12" y1="134.62" x2="58.42" y2="134.62" width="0.1524" layer="91"/>
 <pinref part="VREGIN2" gate="G$1" pin="2"/>
-<wire x1="45.72" y1="134.62" x2="58.42" y2="134.62" width="0.1524" layer="91"/>
-<junction x="58.42" y="134.62"/>
 <junction x="71.12" y="134.62"/>
 <pinref part="5VREG" gate="G$1" pin="GND"/>
-<pinref part="VREGOUT2" gate="G$1" pin="-"/>
-<junction x="45.72" y="134.62"/>
 </segment>
 <segment>
@@
 <wire x1="33.02" y1="144.78" x2="33.02" y2="142.24" width="0.1524" layer="91"/>
 <pinref part="VREGIN2" gate="G$1" pin="1"/>
-<wire x1="33.02" y1="142.24" x2="45.72" y2="142.24" width="0.1524" layer="91"/>
 <junction x="58.42" y="142.24"/>
 <pinref part="5VREG" gate="G$1" pin="IN"/>
-<wire x1="45.72" y1="142.24" x2="58.42" y2="142.24" width="0.1524" layer="91"/>
+<wire x1="33.02" y1="142.24" x2="58.42" y2="142.24" width="0.1524" layer="91"/>
 <wire x1="63.5" y1="142.24" x2="58.42" y2="142.24" width="0.1524" layer="91"/>
-<pinref part="VREGOUT2" gate="G$1" pin="+"/>
-<junction x="45.72" y="142.24"/>
-</segment>
-</net>
+</segment>
+</net>

Commit message: Replaced through hole with smd
Parts:
- C1POWER, VREGIN1: value .1uf -> .1uF; device rcl:C-EU025-025X050 -> rcl:C-EUC0805K
- C3, C4: value 22pf -> 22pF; device rcl:C-EU025-025X050 -> rcl:C-EUC0805K
- LCD_BAK_RES, LCD_POW_RES, RESETPULLUP: device rcl:R-EU_0204/7 -> resistor:R-EU_M0805
- PULLDOWN0: value 30k -> 30K; device rcl:R-EU_0204/7 -> resistor:R-EU_M0805
- PULLDOWN1: value 20k -> 20K; device rcl:R-EU_0204/7 -> resistor:R-EU_M0805
- R12: value 15k -> 15K; device resistor:R-EU_0207/7 -> resistor:R-EU_M0805
- RESETCAP: value .1uf -> 0.33µF; device rcl:C-EU025-025X050 -> rcl:C-EUC0805K
- VREGIN2: device rcl:C-EU025-025X050 -> rcl:C-EUC0805K
Other:
- moved on the sheet: C3, C4, RESETCAP

Commit message: Still working
Parts:
- added J2: AVR_SPI_PROG_5X2PTH2, SparkFun-Connectors:AVR_SPI_PROG_5X2PTH2
- added VREGOUT2: 10uf, resistor:CPOL-EUE2.5-6
- BACKLIGHT_E: value bklight enable -> (none)
- renumbered JP1 to BACKLIGHT_E, R11 to GATE_V
Connections:
- removed net 12V_I/P_TEST: PULLDOWN0.1, PULLDOWN1.2, UC.PB5
- removed net D11: UC.PB3
- removed net D12: UC.PB4
- new net MISO: J2.MISO, UC.PB4
- new net MOSI: J2.MOSI, UC.PB3
- new net PB5/SCK: J2.SCK, PULLDOWN0.1, PULLDOWN1.2, UC.PB5
- net 12V_JACK_INPUT: now also VREGOUT2.+
- net GND: now also J2.GND@1, J2.GND@2, J2.GND@3, J2.GND@4, VREGOUT2.-
- net RESET: now also J2.RESET
Other:
- moved on the sheet: LCD_BAK_RES, LCD_CONTRAST, SUPPLY_JACK

Commit message: Still working
Parts:
- added JP1: (no value), pinhead:PINHD-1X3
- AREF_SET, CURRENT_SET_RES, GATE_V, LCD_CONTRAST, V+_DIVIDER: device rcl:R-TRIMM64W -> pot:TRIM_EU-S64W
- renumbered POW_SLECTION_JUMPER to POW_SELECT, SUPPLY_JACK to 12V
Connections:
- new net N$2: 7812.IN, JP1.1, VREGIN1.1
- net +5V: now also AREF_SET.A, J2.VCC; no longer AREF_SET.E
- net GND: now also AREF_SET.E; no longer AREF_SET.A
- net V+: now also JP1.2; no longer 7812.IN, VREGIN1.1
Other:
- moved on the sheet: RESETPULLUP

Commit message: Still working
Parts:
- added C1POWER1, C1POWER2: .1uF, rcl:C-EUC0805K
- renumbered BACKLIGHT_E to BACKLIGHT, LCD_BAK_RES to BACK_RES, LCD_CONTRAST to CONTRAST
Connections:
- net +5V: now also C1POWER1.1
- net AREF: now also C1POWER2.1
- net GND: now also C1POWER1.2, C1POWER2.2
Changed lines of the file:
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@@
 <layer number="255" name="routoute" color="7" fill="1" visible="yes" active="yes"/>
 </layers>
-<schematic xreflabel="%F%N/%S.%C%R" xrefpart="/%S.%C%R">
+<schematic xreflabel="%F%N/%S" xrefpart="/%S.%C%R">
 <attributes>
 </attributes>
@@
 <part name="LCD_POW_RES" library="resistor" library_urn="urn:adsk.eagle:library:348" deviceset="R-EU_" device="M0805" value="220"/>
 <part name="GND16" library="supply1" deviceset="GND" device=""/>
-<part name="LCD_BAK_RES" library="resistor" library_urn="urn:adsk.eagle:library:348" deviceset="R-EU_" device="M0805" value="220"/>
+<part name="BACK_RES" library="resistor" library_urn="urn:adsk.eagle:library:348" deviceset="R-EU_" device="M0805" value="220"/>
 <part name="GND17" library="supply1" deviceset="GND" device=""/>
-<part name="LCD_CONTRAST" library="pot" library_urn="urn:adsk.eagle:library:331" deviceset="TRIM_EU-" device="S64W" value="50k"/>
+<part name="CONTRAST" library="pot" library_urn="urn:adsk.eagle:library:331" deviceset="TRIM_EU-" device="S64W" value="50k"/>
 <part name="P+15" library="supply1" deviceset="+5V" device=""/>
 <part name="GND18" library="supply1" deviceset="GND" device=""/>
 <part name="P+16" library="supply1" deviceset="+5V" device=""/>
-<part name="BACKLIGHT_E" library="pinhead" deviceset="PINHD-1X2" device=""/>
+<part name="BACKLIGHT" library="pinhead" deviceset="PINHD-1X2" device=""/>
 <part name="GND19" library="supply1" deviceset="GND" device=""/>
 <part name="POW_SELECT" library="pinhead" deviceset="PINHD-1X3" device=""/>
@@
 <part name="JP1" library="pinhead" library_urn="urn:adsk.eagle:library:325" deviceset="PINHD-1X3" device=""/>
 <part name="P+1" library="supply1" deviceset="+5V" device=""/>
+<part name="C1POWER1" library="rcl" library_urn="urn:adsk.eagle:library:334" deviceset="C-EU" device="C0805K" value=".1uF"/>
+<part name="P+9" library="supply1" deviceset="+5V" device=""/>
+<part name="GND25" library="supply1" deviceset="GND" device=""/>
+<part name="C1POWER2" library="rcl" library_urn="urn:adsk.eagle:library:334" deviceset="C-EU" device="C0805K" value=".1uF"/>
+<part name="GND26" library="supply1" deviceset="GND" device=""/>
 </parts>
 <sheets>
@@
 <wire x1="-15.24" y1="45.72" x2="-15.24" y2="43.18" width="0.1524" layer="91"/>
 <wire x1="-10.16" y1="45.72" x2="-15.24" y2="45.72" width="0.1524" layer="91"/>
+<junction x="-15.24" y="45.72"/>
 </segment>
 <segment>
@@
 <attribute name="VALUE" x="-30.48" y="101.6" size="1.778" layer="96"/>
 </instance>
+<instance part="C1POWER1" gate="G$1" x="-12.7" y="55.88"/>
+<instance part="P+9" gate="1" x="-12.7" y="66.04" smashed="yes">
+<attribute name="VALUE" x="-10.16" y="60.96" size="1.778" layer="96" rot="R90"/>
+</instance>
+<instance part="GND25" gate="1" x="-12.7" y="43.18"/>
+<instance part="C1POWER2" gate="G$1" x="111.76" y="83.82"/>
+<instance part="GND26" gate="1" x="111.76" y="73.66"/>
 </instances>
 <busses>
@@
 <pinref part="P+1" gate="1" pin="+5V"/>
 <wire x1="-30.48" y1="104.14" x2="-27.94" y2="104.14" width="0.1524" layer="91"/>
+</segment>
+<segment>
+<pinref part="C1POWER1" gate="G$1" pin="1"/>
+<pinref part="P+9" gate="1" pin="+5V"/>
+<wire x1="-12.7" y1="58.42" x2="-12.7" y2="63.5" width="0.1524" layer="91"/>
 </segment>
 </net>
@@
 <wire x1="124.46" y1="78.74" x2="124.46" y2="81.28" width="0.1524" layer="91"/>
 </segment>
+<segment>
+<pinref part="GND25" gate="1" pin="GND"/>
+<pinref part="C1POWER1" gate="G$1" pin="2"/>
+<wire x1="-12.7" y1="45.72" x2="-12.7" y2="50.8" width="0.1524" layer="91"/>
+</segment>
+<segment>
+<pinref part="C1POWER2" gate="G$1" pin="2"/>
+<pinref part="GND26" gate="1" pin="GND"/>
+<wire x1="111.76" y1="76.2" x2="111.76" y2="78.74" width="0.1524" layer="91"/>
+</segment>
 </net>
 <net name="CRYSTAL1" class="0">
@@
 <segment>
 <pinref part="AREF_SET" gate="1" pin="S"/>
-<wire x1="119.38" y1="86.36" x2="116.84" y2="86.36" width="0.1524" layer="91"/>
-<label x="116.84" y="86.36" size="1.778" layer="95" rot="R180" xref="yes"/>
+<wire x1="119.38" y1="86.36" x2="111.76" y2="86.36" width="0.1524" layer="91"/>
+<label x="106.68" y="86.36" size="1.778" layer="95" rot="R180" xref="yes"/>
+<pinref part="C1POWER2" gate="G$1" pin="1"/>
+<wire x1="111.76" y1="86.36" x2="106.68" y2="86.36" width="0.1524" layer="91"/>
+<junction x="111.76" y="86.36"/>
 </segment>
 </net>
@@
 <instance part="LCD_POW_RES" gate="G$1" x="7.62" y="66.04"/>
 <instance part="GND16" gate="1" x="7.62" y="58.42" rot="R270"/>
-<instance part="LCD_BAK_RES" gate="G$1" x="22.86" y="25.4" rot="R90"/>
+<instance part="BACK_RES" gate="G$1" x="22.86" y="25.4" rot="R90"/>
 <instance part="GND17" gate="1" x="22.86" y="15.24"/>
-<instance part="LCD_CONTRAST" gate="1" x="-36.825290625" y="64.38225" smashed="yes">
+<instance part="CONTRAST" gate="1" x="-36.825290625" y="64.38225" smashed="yes">
 <attribute name="NAME" x="-42.794290625" y="60.57225" size="1.778" layer="95" rot="R90"/>
 <attribute name="VALUE" x="-40.635290625" y="60.57225" size="1.778" layer="96" rot="R90"/>
@@
 <attribute name="VALUE" x="-43.18" y="35.56" size="1.778" layer="96" rot="R180"/>
 </instance>
-<instance part="BACKLIGHT_E" gate="G$1" x="-35.56" y="35.56" smashed="yes" rot="R90">
+<instance part="BACKLIGHT" gate="G$1" x="-35.56" y="35.56" smashed="yes" rot="R90">
 <attribute name="NAME" x="-41.91" y="26.035" size="1.778" layer="95"/>
 <attribute name="VALUE" x="-30.48" y="29.21" size="1.778" layer="96" rot="R90"/>
@@
 </segment>
 <segment>
-<pinref part="LCD_BAK_RES" gate="G$1" pin="1"/>
+<pinref part="BACK_RES" gate="G$1" pin="1"/>
 <pinref part="GND17" gate="1" pin="GND"/>
 <wire x1="22.86" y1="20.32" x2="22.86" y2="17.78" width="0.1524" layer="91"/>
@@
 <segment>
 <pinref part="GND18" gate="1" pin="GND"/>
-<pinref part="LCD_CONTRAST" gate="1" pin="A"/>
+<pinref part="CONTRAST" gate="1" pin="A"/>
 <wire x1="-35.56" y1="58.42" x2="-36.825290625" y2="58.42" width="0.1524" layer="91"/>
 <wire x1="-36.825290625" y1="58.42" x2="-36.825290625" y2="59.30225" width="0.1524" layer="91"/>
@@
 <segment>
 <wire x1="25.4" y1="63.5" x2="-15.24" y2="63.5" width="0.1524" layer="91"/>
-<pinref part="LCD_CONTRAST" gate="1" pin="S"/>
+<pinref part="CONTRAST" gate="1" pin="S"/>
 <wire x1="-31.745290625" y1="64.38225" x2="-15.24" y2="64.38225" width="0.1524" layer="91"/>
 <wire x1="-15.24" y1="64.38225" x2="-15.24" y2="63.5" width="0.1524" layer="91"/>
@@
 <segment>
 <pinref part="P+15" gate="1" pin="+5V"/>
-<pinref part="LCD_CONTRAST" gate="1" pin="E"/>
+<pinref part="CONTRAST" gate="1" pin="E"/>
 <wire x1="-35.56" y1="73.66" x2="-36.825290625" y2="71.12" width="0.1524" layer="91"/>
 <wire x1="-36.825290625" y1="71.12" x2="-36.825290625" y2="69.46225" width="0.1524" layer="91"/>
@@
 <pinref part="P+16" gate="1" pin="+5V"/>
 <wire x1="-45.72" y1="33.02" x2="-38.1" y2="33.02" width="0.1524" layer="91"/>
-<pinref part="BACKLIGHT_E" gate="G$1" pin="1"/>
+<pinref part="BACKLIGHT" gate="G$1" pin="1"/>
 </segment>
 </net>
@@
 <net name="N$14" class="0">
 <segment>
-<pinref part="LCD_BAK_RES" gate="G$1" pin="2"/>
+<pinref part="BACK_RES" gate="G$1" pin="2"/>
 <wire x1="25.4" y1="30.48" x2="22.86" y2="30.48" width="0.1524" layer="91"/>
 <pinref part="LCD1" gate="G$1" pin="K"/>
@@
 <wire x1="25.4" y1="33.02" x2="-35.56" y2="33.02" width="0.1524" layer="91"/>
 <label x="-20.32" y="30.48" size="1.27" layer="95" rot="R270" xref="yes"/>
-<pinref part="BACKLIGHT_E" gate="G$1" pin="2"/>
+<pinref part="BACKLIGHT" gate="G$1" pin="2"/>
 <pinref part="LCD1" gate="G$1" pin="A"/>
 </segment>

Commit message: Complete I guess
Parts:
- 7805: value 7805 -> 5V
- renumbered 5VREG to 7805, AREF_SET to AREF, BACK_RES to R15, C1POWER to C9, C1POWER1 to C8, C1POWER2 to C11, CONTRAST to CONT, CURRENT_SET_RES to CURRENT_SET, IC1 to OPAMP, J1 to FTDI, J2 to ASP, JP1 to V+TO12, LCD1 to LCD, LCD_POW_RES to R16, PULLDOWN0 to R14, PULLDOWN1 to R13, RESETCAP to C10, RESETPULLUP to R17, UC to ATMEGA328P, V+_DIVIDER to V+, VREGIN1 to C6, VREGIN2 to C13, VREGOUT to C12, VREGOUT1 to C5, VREGOUT2 to C7, X1 to LOAD

Commit message: Before moving HS and Pot
Other:
- note removed: "Rev 3: Atmega with ftdi and arduino bootloader"
Changed lines of the file:
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@@
 <grid distance="0.01" unitdist="inch" unit="inch" style="lines" multiple="1" display="no" altdistance="0.01" altunitdist="inch" altunit="inch"/>
 <layers>
-<layer number="1" name="Top" color="4" fill="1" visible="yes" active="no"/>
-<layer number="2" name="Route2" color="1" fill="3" visible="yes" active="no"/>
-<layer number="3" name="Route3" color="4" fill="3" visible="yes" active="no"/>
-<layer number="4" name="Route4" color="1" fill="4" visible="yes" active="no"/>
-<layer number="5" name="Route5" color="4" fill="4" visible="yes" active="no"/>
-<layer number="6" name="Route6" color="1" fill="8" visible="yes" active="no"/>
-<layer number="7" name="Route7" color="4" fill="8" visible="yes" active="no"/>
-<layer number="8" name="Route8" color="1" fill="2" visible="yes" active="no"/>
-<layer number="9" name="Route9" color="4" fill="2" visible="yes" active="no"/>
-<layer number="10" name="Route10" color="1" fill="7" visible="yes" active="no"/>
-<layer number="11" name="Route11" color="4" fill="7" visible="yes" active="no"/>
-<layer number="12" name="Route12" color="1" fill="5" visible="yes" active="no"/>
-<layer number="13" name="Route13" color="4" fill="5" visible="yes" active="no"/>
-<layer number="14" name="Route14" color="1" fill="6" visible="yes" active="no"/>
-<layer number="15" name="Route15" color="4" fill="6" visible="yes" active="no"/>
-<layer number="16" name="Bottom" color="1" fill="1" visible="yes" active="no"/>
-<layer number="17" name="Pads" color="2" fill="1" visible="yes" active="no"/>
-<layer number="18" name="Vias" color="2" fill="1" visible="yes" active="no"/>
-<layer number="19" name="Unrouted" color="6" fill="1" visible="yes" active="no"/>
-<layer number="20" name="Dimension" color="15" fill="1" visible="yes" active="no"/>
-<layer number="21" name="tPlace" color="16" fill="1" visible="yes" active="no"/>
-<layer number="22" name="bPlace" color="14" fill="1" visible="yes" active="no"/>
-<layer number="23" name="tOrigins" color="15" fill="1" visible="yes" active="no"/>
-<layer number="24" name="bOrigins" color="15" fill="1" visible="yes" active="no"/>
-<layer number="25" name="tNames" color="7" fill="1" visible="yes" active="no"/>
-<layer number="26" name="bNames" color="7" fill="1" visible="yes" active="no"/>
-<layer number="27" name="tValues" color="7" fill="1" visible="yes" active="no"/>
-<layer number="28" name="bValues" color="7" fill="1" visible="yes" active="no"/>
+<layer number="1" name="Top" color="4" fill="1" visible="no" active="no"/>
+<layer number="2" name="Route2" color="1" fill="3" visible="no" active="no"/>
+<layer number="3" name="Route3" color="4" fill="3" visible="no" active="no"/>
+<layer number="4" name="Route4" color="1" fill="4" visible="no" active="no"/>
+<layer number="5" name="Route5" color="4" fill="4" visible="no" active="no"/>
+<layer number="6" name="Route6" color="1" fill="8" visible="no" active="no"/>
+<layer number="7" name="Route7" color="4" fill="8" visible="no" active="no"/>
+<layer number="8" name="Route8" color="1" fill="2" visible="no" active="no"/>
+<layer number="9" name="Route9" color="4" fill="2" visible="no" active="no"/>
+<layer number="10" name="Route10" color="1" fill="7" visible="no" active="no"/>
+<layer number="11" name="Route11" color="4" fill="7" visible="no" active="no"/>
+<layer number="12" name="Route12" color="1" fill="5" visible="no" active="no"/>
+<layer number="13" name="Route13" color="4" fill="5" visible="no" active="no"/>
+<layer number="14" name="Route14" color="1" fill="6" visible="no" active="no"/>
+<layer number="15" name="Route15" color="4" fill="6" visible="no" active="no"/>
+<layer number="16" name="Bottom" color="1" fill="1" visible="no" active="no"/>
+<layer number="17" name="Pads" color="2" fill="1" visible="no" active="no"/>
+<layer number="18" name="Vias" color="2" fill="1" visible="no" active="no"/>
+<layer number="19" name="Unrouted" color="6" fill="1" visible="no" active="no"/>
+<layer number="20" name="Dimension" color="15" fill="1" visible="no" active="no"/>
+<layer number="21" name="tPlace" color="16" fill="1" visible="no" active="no"/>
+<layer number="22" name="bPlace" color="14" fill="1" visible="no" active="no"/>
+<layer number="23" name="tOrigins" color="15" fill="1" visible="no" active="no"/>
+<layer number="24" name="bOrigins" color="15" fill="1" visible="no" active="no"/>
+<layer number="25" name="tNames" color="7" fill="1" visible="no" active="no"/>
+<layer number="26" name="bNames" color="7" fill="1" visible="no" active="no"/>
+<layer number="27" name="tValues" color="7" fill="1" visible="no" active="no"/>
+<layer number="28" name="bValues" color="7" fill="1" visible="no" active="no"/>
 <layer number="29" name="tStop" color="7" fill="3" visible="no" active="no"/>
 <layer number="30" name="bStop" color="7" fill="6" visible="no" active="no"/>
@@
 <layer number="35" name="tGlue" color="7" fill="4" visible="no" active="no"/>
 <layer number="36" name="bGlue" color="7" fill="5" visible="no" active="no"/>
-<layer number="37" name="tTest" color="7" fill="1" visible="yes" active="no"/>
-<layer number="38" name="bTest" color="7" fill="1" visible="yes" active="no"/>
+<layer number="37" name="tTest" color="7" fill="1" visible="no" active="no"/>
+<layer number="38" name="bTest" color="7" fill="1" visible="no" active="no"/>
 <layer number="39" name="tKeepout" color="4" fill="11" visible="no" active="no"/>
 <layer number="40" name="bKeepout" color="1" fill="11" visible="no" active="no"/>
@@
 <layer number="44" name="Drills" color="7" fill="1" visible="no" active="no"/>
 <layer number="45" name="Holes" color="7" fill="1" visible="no" active="no"/>
-<layer number="46" name="Milling" color="3" fill="1" visible="yes" active="no"/>
-<layer number="47" name="Measures" color="7" fill="1" visible="yes" active="no"/>
-<layer number="48" name="Document" color="7" fill="1" visible="yes" active="no"/>
-<layer number="49" name="Reference" color="7" fill="1" visible="yes" active="no"/>
-<layer number="50" name="dxf" color="7" fill="1" visible="yes" active="no"/>
-<layer number="51" name="tDocu" color="6" fill="1" visible="yes" active="no"/>
-<layer number="52" name="bDocu" color="7" fill="1" visible="yes" active="no"/>
-<layer number="53" name="tGND_GNDA" color="7" fill="9" visible="yes" active="no"/>
-<layer number="54" name="bGND_GNDA" color="1" fill="9" visible="yes" active="no"/>
-<layer number="56" name="wert" color="7" fill="1" visible="yes" active="no"/>
-<layer number="57" name="tCAD" color="7" fill="1" visible="yes" active="no"/>
-<layer number="59" name="tCarbon" color="7" fill="1" visible="yes" active="no"/>
-<layer number="60" name="bCarbon" color="7" fill="1" visible="yes" active="no"/>
+<layer number="46" name="Milling" color="3" fill="1" visible="no" active="no"/>
+<layer number="47" name="Measures" color="7" fill="1" visible="no" active="no"/>
+<layer number="48" name="Document" color="7" fill="1" visible="no" active="no"/>
+<layer number="49" name="Reference" color="7" fill="1" visible="no" active="no"/>
+<layer number="50" name="dxf" color="7" fill="1" visible="no" active="no"/>
+<layer number="51" name="tDocu" color="6" fill="1" visible="no" active="no"/>
+<layer number="52" name="bDocu" color="7" fill="1" visible="no" active="no"/>
+<layer number="53" name="tGND_GNDA" color="7" fill="9" visible="no" active="no"/>
+<layer number="54" name="bGND_GNDA" color="1" fill="9" visible="no" active="no"/>
+<layer number="56" name="wert" color="7" fill="1" visible="no" active="no"/>
+<layer number="57" name="tCAD" color="7" fill="1" visible="no" active="no"/>
+<layer number="59" name="tCarbon" color="7" fill="1" visible="no" active="no"/>
+<layer number="60" name="bCarbon" color="7" fill="1" visible="no" active="no"/>
 <layer number="90" name="Modules" color="5" fill="1" visible="yes" active="yes"/>
 <layer number="91" name="Nets" color="2" fill="1" visible="yes" active="yes"/>
@@
 <sheet>
 <plain>
-<text x="83.82" y="2.54" size="1.778" layer="91">Rev 3:
-Atmega with ftdi and arduino bootloader</text>
 </plain>
 <instances>
@@
 </segment>
 </net>
-<net name="N$3" class="0">
-<segment>
-<wire x1="83.82" y1="0" x2="83.82" y2="7.62" width="0.1524" layer="91"/>
-<wire x1="83.82" y1="7.62" x2="134.62" y2="7.62" width="0.1524" layer="91"/>
-<wire x1="134.62" y1="7.62" x2="134.62" y2="0" width="0.1524" layer="91"/>
-<wire x1="134.62" y1="0" x2="83.82" y2="0" width="0.1524" layer="91"/>
-</segment>
-</net>
 <net name="+12V" class="0">
 <segment>
@@
 </drawing>
 <compatibility>
-<note version="6.3" minversion="6.2.2" severity="warning">
-Since Version 6.2.2 text objects can contain more than one line,
-which will not be processed correctly with this version.
-</note>
 <note version="8.2" severity="warning">
 Since Version 8.2, Eagle supports online libraries. The ids
